File: hachidori-esp/hachidori.sch (KiCad schematic (older format))
At the start: 80 parts, among them CON1 microUSB_CONSOLE, P1 VIN, P10 PWM1, P11 PWM2, P12 PWM3, P2 UART, P3 ADC, P4 I2C, P5 M3, P6 M2, P7 M1, P8 M0, P9 PWM0, Q1 BSS138, Q2 BSS138, Q3 BSS138, Q4 BSS138, SW1 FLASH, SW2 RESET, U1 AP7661-33ER, U2 MPU-9250, U3 ESP-13-WROOM-02, U4 BME280, U5 PCA9685, U6 FT230X, U7 INA226

Commit message: modified
Parts:
- added LED4, LED5: Front, droneworks:LED_1608mm, symbol LED
- added LED6, LED7: Back, droneworks:LED_1608mm, symbol LED
- added P13: SW-UART, droneworks:Pin_Header_1x03, symbol CONN_01X03
- added R28, R29, R30, R31: 220, rohm:MCR03, symbol R
- added TH4: GPIO, droneworks:TH, symbol throughhole
- LED2: value RXLED -> RX
- LED3: value TXLED -> TX
- Q1, Q2, Q3, Q4: value BSS138 -> IRLML6344TRPBF
- U1: value AP7661-33ER -> NCP1117ST33
Connections:
- net 3V3: now also U7.1 (A1), R28.1, R29.1, R30.1, R31.1; no longer R14.2, R15.2, U6.3 (VCCIO)
- net GND: now also LED4.1 (K), LED5.1 (K), LED6.1 (K), LED7.1 (K); no longer U7.1 (A1)
- net TOUT: now also R6.1, R8.2, U3.16 (TOUT); no longer P3.2 (P2), R6.2
- net GPIO: now reaches U3.17 (GPIO16)
- net GPIO: now also TH4.1
- net FTDI-3V3: now reaches CB9.1, U6.10 (3v3OUT), U6.11 (~Reset)
- net FTDI-3V3: now also R14.2, R15.2, U6.3 (VCCIO)
- net RXD renamed ESP-TXD
- removed net TXD: P2.2 (P2), U3.11 (RXD), U6.1 (TxD)
- new net: LED4.2 (A), R28.2
- new net: LED5.2 (A), R29.2
- new net: LED6.2 (A), R30.2
- new net: LED7.2 (A), R31.2
- new net ESP-RXD: P13.2 (P2), U3.11 (RXD)
- new net ESP-RXDpin: P13.1 (P1), P2.2 (P2)
- new net FTDI-TXD: P13.3 (P3), U6.1 (TxD)
- new net TOUTpin: P3.2 (P2), R6.2
- no-connect marks 21 -> 20
Other:
- note added: "ESP-RXD"
- note added: "ESP-TXDpin"
- note added: "FTDI-RXD"
- note added: "FTDI-TXD"
- note added: "RXDpin"
- note added: "SW-UART pin header\nUse UARTpin -> 1-2pin\nUse FTDI -> 2-3pin"
- note removed: "ESP_RXD"
- note removed: "ESP_TXD"
- note removed: "TOUT"
- moved on the sheet: CB3, CB6, CB8, CB9, CC1, CC2, CE1, CE3, CON1, D1, D2, D3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
