File: esp32-dev-board/hachidori.sch (KiCad schematic (older format))
At the start: 35 parts, among them P1 VIN, P2 GPIO, P3 I2C, P4 SERVO, P5 GPIO, P8 Program, SW1 RESET, SW2 FLASH, U1 ADP3338, U2 INA226, U3 ESP-WROOM-32

Commit message: fix
Parts:
- removed CB6: 104, droneworks:GRM18, symbol C
Changed lines of the file:
@@
-$EndComp
-$Comp
-L C CB6
-U 1 1 57B915F7
-P 9300 5350
-F 0 "CB6" H 9325 5450 50  0000 L CNN
-F 1 "104" H 9325 5250 50  0000 L CNN
-F 2 "droneworks:GRM18" H 9338 5200 50  0001 C CNN
-F 3 "" H 9300 5350 50  0000 C CNN
-	1    9300 5350
-	1    0    0    -1
 $EndComp
 $Comp
@@
 Wire Wire Line
 	3650 2450 3650 2250
-Wire Wire Line
-	9300 5650 9300 5500
-Wire Wire Line
-	9300 1700 9300 5200
 Connection ~ 5100 5650
 Wire Wire Line
@@
 	4950 2900 5650 2900
 Wire Wire Line
-	2750 5650 9300 5650
-Wire Wire Line
 	2200 1700 2200 5050
 Wire Wire Line
@@
 	9550 3100 9150 3100
 Connection ~ 9150 3100
-Connection ~ 9150 5650
 Wire Wire Line
 	7450 5650 7450 5600
@@
 Wire Wire Line
 	3950 3300 5650 3300
-Connection ~ 4500 5250
 $Comp
 L PICOLED-RGB D1
@@
 Wire Wire Line
 	8300 5000 9300 5000
-Connection ~ 9300 5000
 Wire Wire Line
 	7000 5200 7200 5200
@@
 	1    0    0    -1
 $EndComp
+Wire Wire Line
+	2750 5650 9150 5650
+Wire Wire Line
+	9300 5000 9300 1700
 $EndSCHEMATC

Commit message: fix
Parts:
- removed P8: Program, droneworks:Pin_Header_1x05, symbol CONN_01X05
- added P6: 3V3_GND, droneworks:Pin_Header_1x02, symbol CONN_01X02
- added P7: Program, droneworks:Pin_Header_1x02, symbol CONN_01X02
Connections:
- net 3V3: now also P2.7 (P7), P6.1 (P1)
- net GND: now also P6.2 (P2); no longer P2.7 (P7)
- net RXD0: now also P7.2 (P2)
- net TXD0: now also P7.1 (P1)
Changed lines of the file:
@@
 Sheet 1 1
 Title "hachidori-32"
-Date "2017-02-17"
-Rev "0.11"
+Date "2017-02-24"
+Rev "0.12"
 Comp ""
 Comment1 "Copyright (c) 2017 DroneWorks Inc."
@@
 Text Label 3950 3900 0    60   ~ 0
 CH3
-$Comp
-L CONN_01X05 P8
-U 1 1 58A39F84
-P 9750 2900
-F 0 "P8" H 9750 3200 50  0000 C CNN
-F 1 "Program" V 9850 2900 50  0000 C CNN
-F 2 "droneworks:Pin_Header_1x05" H 9750 2900 50  0001 C CNN
-F 3 "" H 9750 2900 50  0000 C CNN
-	1    9750 2900
-	1    0    0    -1
-$EndComp
 Text Notes 9350 2700 0    60   ~ 0
 GND
-Text Notes 9350 3100 0    60   ~ 0
-GND
-Text Notes 9350 2900 0    60   ~ 0
+Text Notes 9350 2600 0    60   ~ 0
 3V3
-Text Notes 9350 2800 0    60   ~ 0
+Text Notes 9350 2850 0    60   ~ 0
 TXD
-Text Notes 9350 3000 0    60   ~ 0
+Text Notes 9350 2950 0    60   ~ 0
 RXD
 Text Label 7700 3000 0    60   ~ 0
@@
 	7650 2700 9550 2700
 Wire Wire Line
-	9150 2700 9150 5650
+	9150 5650 9150 2700
 Wire Wire Line
 	7100 5600 7100 5700
@@
 	7650 3000 8300 3000
 Wire Wire Line
-	8300 3000 8300 2800
-Wire Wire Line
-	9550 2900 9300 2900
-Connection ~ 9300 2900
-Wire Wire Line
-	9550 3100 9150 3100
-Connection ~ 9150 3100
+	8300 3000 8300 2850
 Wire Wire Line
 	7450 5650 7450 5600
@@
 Wire Wire Line
 	5650 3000 3950 3000
-Text Notes 3950 2900 0    60   ~ 0
-GND
 $Comp
 L CONN_01X03 P3
@@
 $EndComp
 Wire Wire Line
-	3950 2900 4350 2900
-Connection ~ 4350 2900
-Wire Wire Line
 	3950 3300 5650 3300
 $Comp
@@
 	7100 4250 7100 5000
 Wire Wire Line
-	8300 5000 9300 5000
+	9300 5000 8300 5000
 Wire Wire Line
 	7000 5200 7200 5200
@@
 	7650 2900 8500 2900
 Wire Wire Line
-	8300 2800 9550 2800
-Wire Wire Line
-	9550 3000 8400 3000
-Wire Wire Line
-	8400 3000 8400 3100
+	8300 2850 9550 2850
+Wire Wire Line
+	9550 2950 8400 2950
+Wire Wire Line
+	8400 2950 8400 3100
 Wire Wire Line
 	8400 3100 7650 3100
@@
 	2750 5650 9150 5650
 Wire Wire Line
-	9300 5000 9300 1700
+	9300 1700 9300 5000
+Connection ~ 9300 2600
+Wire Wire Line
+	9550 2600 9300 2600
+$Comp
+L CONN_01X02 P7
+U 1 1 58AC5648
+P 9750 2900
+F 0 "P7" H 9750 3050 50  0000 C CNN
+F 1 "Program" V 9850 2900 50  0000 C CNN
+F 2 "droneworks:Pin_Header_1x02" H 9750 2900 50  0001 C CNN
+F 3 "" H 9750 2900 50  0000 C CNN
+	1    9750 2900
+	1    0    0    -1
+$EndComp
+$Comp
+L CONN_01X02 P6
+U 1 1 58AC56CB
+P 9750 2650
+F 0 "P6" H 9750 2800 50  0000 C CNN
+F 1 "3V3_GND" V 9850 2650 50  0000 C CNN
+F 2 "droneworks:Pin_Header_1x02" H 9750 2650 50  0001 C CNN
+F 3 "" H 9750 2650 50  0000 C CNN
+	1    9750 2650
+	1    0    0    -1
+$EndComp
+Text Notes 3950 2900 0    60   ~ 0
+3V3
+Wire Wire Line
+	3950 2900 4500 2900
+Connection ~ 4500 2900
 $EndSCHEMATC
